Commit message: fix

File: src/gld_robot_description/model/gld_robot_description.urdf (robot description, URDF)
Before this commit: robot gld_robot_description, 10 links, 9 joints
Links:
- removed link base_footprint
- removed link chassis
- removed link livox_frame
- added link base
- added link livox
Joints:
- removed joint base_to_chassis
- removed joint chassis_to_D405_1
- removed joint chassis_to_D405_2
- removed joint chassis_to_D456_1
- removed joint chassis_to_D456_2
- removed joint chassis_to_livox_frame
- removed joint chassis_to_orbbec_gemini_1
- removed joint chassis_to_orbbec_gemini_2
- removed joint chassis_to_orbbec_gemini_3
- added joint base_to_D405_1: type fixed, parent base, child D405_1_link, origin xyz=0.0 0.0 0.0 rpy=0 0 0
- added joint base_to_D405_2: type fixed, parent base, child D405_2_link, origin xyz=0.0 0.0 0.0 rpy=0 0 0
- added joint base_to_D456_1: type fixed, parent base, child D456_1_link, origin xyz=0.0 0.0 0.0 rpy=0 0 0
- added joint base_to_D456_2: type fixed, parent base, child D456_2_link, origin xyz=0.0 0.0 0.0 rpy=0 0 0
- added joint base_to_livox: type fixed, parent base, child livox, origin xyz=0.0 0.0 0.0 rpy=0 0 0
- added joint base_to_orbbec_gemini_1: type fixed, parent base, child orbbec_gemini_1_link, origin xyz=0.0 0.0 0.0 rpy=0 0 0
- added joint base_to_orbbec_gemini_2: type fixed, parent base, child orbbec_gemini_2_link, origin xyz=0.0 0.0 0.0 rpy=0 0 0
- added joint base_to_orbbec_gemini_3: type fixed, parent base, child orbbec_gemini_3_link, origin xyz=0.0 0.0 0.0 rpy=0 0 0
